Commit message: Model the car at the width it actually is
gb_ego_width_m was 0.4 against a car that measures 0.28 - which
albomb_core.xacro now agrees with: wheel_track 0.235 + wheel_length 0.04.
The extra 12 cm was hidden padding, and it made every clearance number in
the state machine mean something other than what it said. free_dist in
_check_free_frenet is the gap between the car's side and the obstacle's
edge, so it should be that gap.

_check_close_to_raceline reads the same parameter, which is why an earlier
note said not to touch it. That turns out to be wrong in practice: its only
caller passes an explicit 0.05, so the gb_ego_width_m branch never runs.

The change cuts both ways and the second direction is easy to miss. The
same free check also decides whether the RACELINE is blocked, and a
narrower car is judged blocked less often - so on its own this would make
the car notice obstacles later, not earlier. lateral_width_gb_m takes the
6 cm per side back, 0.3 -> 0.36.

lateral_width_m goes 0.02 -> 0.05 for the same reason in reverse: it is a
real margin now rather than a number compensating for padding elsewhere,
and 5 cm is about what localisation error and the obstacle's measured edge
are worth together. The floor it puts on evasion_distance is 0.19, so the
0.24 in perception.yaml now has 5 cm of slack instead of 2.

Separately: the urdf's wheel_base moved 0.324 -> 0.327 without vesc.yaml
and controller.yaml following. Those three invert the same bicycle model
and a mismatch steers the car to a curvature it is not reporting, so they
move together here.

Co-Authored-By: Claude Opus 5 <noreply@anthropic.com>

File: src/albomb_description/urdf/albomb_core.xacro (robot description, xacro)
@@ -3,7 +3,7 @@
   <xacro:property name="car_name" value="ego_racecar" />
   <xacro:property name="wheel_track" value="0.235" />     <!-- 윤거 -->
-  <xacro:property name="wheel_base" value="0.327" />      <!-- 축거 -->
+  <xacro:property name="wheel_base" value="0.324" />      <!-- 축거 -->
   <xacro:property name="wheel_radius" value="0.05" />     <!-- 바퀴 반지름 -->
-  <xacro:property name="wheel_length" value="0.04" />    <!-- 바퀴 두께 -->
+  <xacro:property name="wheel_length" value="0.045" />    <!-- 바퀴 두께 -->
   <material name="Black">
     <color rgba="0.0 0.0 0.0 1.0"/>
